File: led/led-sheet.kicad_sch (KiCad schematic)
At the start: 3 parts

Commit message: led
Parts:
- removed TP1, TP2: TestPoint, TestPoint:TestPoint_Pad_1.0x1.0mm, symbol Connector:TestPoint
- added Q1: Q_NMOS_DGS, Package_TO_SOT_SMD:SOT-23, symbol Device:Q_NMOS_DGS
- added R1: R, Resistor_SMD:R_0805_2012Metric, symbol Device:R
Connections:
- net LED_A: no longer names the net of D1.2 (A)
- net LED_A: now also R1.2
- net LED_C renamed switched
- net switched: now also Q1.1 (D)
- new net +3V3: R1.1
- new net GND: Q1.3 (S)
- new net control: Q1.2 (G)
Other:
- moved on the sheet: D1
Changed lines of the file:
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@@
 (kicad_sch (version 20201015) (generator eeschema)
   (paper "A4")
-  (junction (at 152.4 83.82) (diameter 0.9144) (color 0 0 0 0))
-  (junction (at 152.4 91.44) (diameter 0.9144) (color 0 0 0 0))
-  (wire (pts (xy 146.05 83.82) (xy 152.4 83.82))
+  (wire (pts (xy 146.05 102.87) (xy 154.305 102.87))
     (stroke (width 0) (type solid) (color 0 0 0 0))
   )
-  (wire (pts (xy 146.05 91.44) (xy 152.4 91.44))
+  (wire (pts (xy 148.59 80.01) (xy 148.59 76.2))
     (stroke (width 0) (type solid) (color 0 0 0 0))
   )
-  (wire (pts (xy 152.4 81.28) (xy 152.4 83.82))
+  (wire (pts (xy 160.02 80.01) (xy 148.59 80.01))
     (stroke (width 0) (type solid) (color 0 0 0 0))
   )
-  (wire (pts (xy 152.4 91.44) (xy 152.4 95.25))
+  (wire (pts (xy 161.29 92.075) (xy 161.29 92.71))
     (stroke (width 0) (type solid) (color 0 0 0 0))
   )
-  (hierarchical_label "LED_A" (shape input) (at 146.05 83.82 180)
+  (wire (pts (xy 161.925 97.79) (xy 169.545 97.79))
+    (stroke (width 0) (type solid) (color 0 0 0 0))
+  )
+  (wire (pts (xy 161.925 107.95) (xy 161.925 111.125))
+    (stroke (width 0) (type solid) (color 0 0 0 0))
+  )
+  (wire (pts (xy 161.925 111.125) (xy 171.45 111.125))
+    (stroke (width 0) (type solid) (color 0 0 0 0))
+  )
+  (wire (pts (xy 167.64 80.01) (xy 176.53 80.01))
+    (stroke (width 0) (type solid) (color 0 0 0 0))
+  )
+  (wire (pts (xy 176.53 80.01) (xy 176.53 85.09))
+    (stroke (width 0) (type solid) (color 0 0 0 0))
+  )
+  (wire (pts (xy 176.53 92.71) (xy 161.29 92.71))
+    (stroke (width 0) (type solid) (color 0 0 0 0))
+  )
+  (wire (pts (xy 179.705 120.015) (xy 190.5 120.015))
+    (stroke (width 0) (type solid) (color 0 0 0 0))
+  )
+  (wire (pts (xy 190.5 120.015) (xy 190.5 123.825))
+    (stroke (width 0) (type solid) (color 0 0 0 0))
+  )
+  (label "switched" (at 164.465 97.79 180)
+    (effects (font (size 1.27 1.27)) (justify right bottom))
+  )
+  (label "switched" (at 169.545 92.71 180)
+    (effects (font (size 1.27 1.27)) (justify right bottom))
+  )
+  (label "ground" (at 170.18 111.125 180)
+    (effects (font (size 1.27 1.27)) (justify right bottom))
+  )
+  (label "ground" (at 186.69 120.015 180)
+    (effects (font (size 1.27 1.27)) (justify right bottom))
+  )
+  (hierarchical_label "control" (shape input) (at 146.05 102.87 180)
     (effects (font (size 1.27 1.27)) (justify right))
   )
-  (hierarchical_label "LED_C" (shape input) (at 146.05 91.44 180)
-    (effects (font (size 1.27 1.27)) (justify right))
-  )
-  (symbol (lib_id "Connector:TestPoint") (at 152.4 81.28 0) (unit 1)
+  (symbol (lib_id "power:+3V3") (at 148.59 76.2 0)
     (in_bom yes) (on_board yes)
-    (property "Reference" "TP1" (id 0) (at 154.94 78.74 0)
-      (effects (font (size 1.27 1.27)) (justify left))
-    )
-    (property "Value" "TestPoint" (id 1) (at 154.94 81.28 0)
-      (effects (font (size 1.27 1.27)) (justify left))
-    )
-    (property "Footprint" "TestPoint:TestPoint_Pad_1.0x1.0mm" (id 2) (at 157.48 81.28 0)
+    (property "Reference" "#PWR05" (id 0) (at 148.59 80.01 0)
       (effects (font (size 1.27 1.27)) hide)
     )
-    (property "Datasheet" "~" (id 3) (at 157.48 81.28 0)
+    (property "Value" "+3V3" (id 1) (at 149.225 70.485 0))
+    (property "Footprint" "" (id 2) (at 148.59 76.2 0)
+      (effects (font (size 1.27 1.27)) hide)
+    )
+    (property "Datasheet" "" (id 3) (at 148.59 76.2 0)
       (effects (font (size 1.27 1.27)) hide)
     )
   )
-  (symbol (lib_id "Connector:TestPoint") (at 152.4 95.25 180) (unit 1)
+  (symbol (lib_id "power:GND") (at 190.5 123.825 0)
     (in_bom yes) (on_board yes)
-    (property "Reference" "TP2" (id 0) (at 154.94 96.52 0)
-      (effects (font (size 1.27 1.27)) (justify right))
-    )
-    (property "Value" "TestPoint" (id 1) (at 154.94 99.06 0)
-      (effects (font (size 1.27 1.27)) (justify right))
-    )
-    (property "Footprint" "TestPoint:TestPoint_Pad_1.0x1.0mm" (id 2) (at 147.32 95.25 0)
+    (property "Reference" "#PWR06" (id 0) (at 190.5 130.175 0)
       (effects (font (size 1.27 1.27)) hide)
     )
-    (property "Datasheet" "~" (id 3) (at 147.32 95.25 0)
+    (property "Value" "GND" (id 1) (at 191.77 128.27 0))
+    (property "Footprint" "" (id 2) (at 190.5 123.825 0)
+      (effects (font (size 1.27 1.27)) hide)
+    )
+    (property "Datasheet" "" (id 3) (at 190.5 123.825 0)
       (effects (font (size 1.27 1.27)) hide)
     )
   )
-  (symbol (lib_id "Device:LED") (at 152.4 87.63 90) (unit 1)
+  (symbol (lib_id "Device:R") (at 163.83 80.01 90)
     (in_bom yes) (on_board yes)
-    (property "Reference" "D1" (id 0) (at 156.21 87.63 90)
+    (property "Reference" "R1" (id 0) (at 164.465 73.66 90))
+    (property "Value" "R" (id 1) (at 164.465 76.2 90))
+    (property "Footprint" "Resistor_SMD:R_0805_2012Metric" (id 2) (at 163.83 81.788 90)
+      (effects (font (size 1.27 1.27)) hide)
+    )
+    (property "Datasheet" "~" (id 3) (at 163.83 80.01 0)
+      (effects (font (size 1.27 1.27)) hide)
+    )
+  )
+  (symbol (lib_id "Device:LED") (at 176.53 88.9 90)
+    (in_bom yes) (on_board yes)
+    (property "Reference" "D1" (id 0) (at 180.34 88.9 90)
       (effects (font (size 1.27 1.27)) (justify right))
     )
-    (property "Value" "LED" (id 1) (at 156.21 90.17 90)
+    (property "Value" "LED" (id 1) (at 180.34 91.44 90)
       (effects (font (size 1.27 1.27)) (justify right))
     )
-    (property "Footprint" "LED_SMD:LED_0805_2012Metric" (id 2) (at 152.4 87.63 0)
+    (property "Footprint" "LED_SMD:LED_0805_2012Metric" (id 2) (at 176.53 88.9 0)
       (effects (font (size 1.27 1.27)) hide)
     )
-    (property "Datasheet" "~" (id 3) (at 152.4 87.63 0)
+    (property "Datasheet" "~" (id 3) (at 176.53 88.9 0)
       (effects (font (size 1.27 1.27)) hide)
     )
+  )
+  (symbol (lib_id "Device:Q_NMOS_DGS") (at 159.385 102.87 0)
+    (in_bom yes) (on_board yes)
+    (property "Reference" "Q1" (id 0) (at 165.1 102.235 0)
+      (effects (font (size 1.27 1.27)) (justify left))
+    )
+    (property "Value" "Q_NMOS_DGS" (id 1) (at 165.1 104.775 0)
+      (effects (font (size 1.27 1.27)) (justify left))
+    )
+    (property "Footprint" "Package_TO_SOT_SMD:SOT-23" (id 2) (at 164.465 100.33 0)
+      (effects (font (size 1.27 1.27)) hide)
+    )
+    (property "Datasheet" "~" (id 3) (at 159.385 102.87 0)
+      (effects (font (size 1.27 1.27)) hide)
+    )

Commit message: net
Parts:
- renumbered D1 to D2, Q1 to Q2, R1 to R2
Changed lines of the file:
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@@
   (symbol (lib_id "power:+3V3") (at 148.59 76.2 0)
     (in_bom yes) (on_board yes)
-    (property "Reference" "#PWR05" (id 0) (at 148.59 80.01 0)
+    (property "Reference" "#PWR07" (id 0) (at 148.59 80.01 0)
       (effects (font (size 1.27 1.27)) hide)
     )
@@
   (symbol (lib_id "power:GND") (at 190.5 123.825 0)
     (in_bom yes) (on_board yes)
-    (property "Reference" "#PWR06" (id 0) (at 190.5 130.175 0)
+    (property "Reference" "#PWR08" (id 0) (at 190.5 130.175 0)
       (effects (font (size 1.27 1.27)) hide)
     )
@@
   (symbol (lib_id "Device:R") (at 163.83 80.01 90)
     (in_bom yes) (on_board yes)
-    (property "Reference" "R1" (id 0) (at 164.465 73.66 90))
+    (property "Reference" "R2" (id 0) (at 164.465 73.66 90))
     (property "Value" "R" (id 1) (at 164.465 76.2 90))
     (property "Footprint" "Resistor_SMD:R_0805_2012Metric" (id 2) (at 163.83 81.788 90)
@@
   (symbol (lib_id "Device:LED") (at 176.53 88.9 90)
     (in_bom yes) (on_board yes)
-    (property "Reference" "D1" (id 0) (at 180.34 88.9 90)
+    (property "Reference" "D2" (id 0) (at 180.34 88.9 90)
       (effects (font (size 1.27 1.27)) (justify right))
     )
@@
   (symbol (lib_id "Device:Q_NMOS_DGS") (at 159.385 102.87 0)
     (in_bom yes) (on_board yes)
-    (property "Reference" "Q1" (id 0) (at 165.1 102.235 0)
+    (property "Reference" "Q2" (id 0) (at 165.1 102.235 0)
       (effects (font (size 1.27 1.27)) (justify left))
     )
