File: led/led-sheet.kicad_sch (KiCad schematic)
At the start: 3 parts, among them Q2 Q_NMOS_DGS

Commit message: baseline
Parts:
- renumbered D2 to D1, Q2 to Q1, R2 to R1
Changed lines of the file:
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@@
 (kicad_sch (version 20201015) (generator eeschema)
   (paper "A4")
+  (junction (at 152.654 80.01) (diameter 0.9144) (color 0 0 0 0))
+  (junction (at 186.944 121.666) (diameter 0.9144) (color 0 0 0 0))
   (wire (pts (xy 146.05 102.87) (xy 154.305 102.87))
     (stroke (width 0) (type solid) (color 0 0 0 0))
@@
     (stroke (width 0) (type solid) (color 0 0 0 0))
   )
-  (wire (pts (xy 160.02 80.01) (xy 148.59 80.01))
+  (wire (pts (xy 152.654 78.486) (xy 152.654 80.01))
+    (stroke (width 0) (type solid) (color 0 0 0 0))
+  )
+  (wire (pts (xy 152.654 80.01) (xy 148.59 80.01))
+    (stroke (width 0) (type solid) (color 0 0 0 0))
+  )
+  (wire (pts (xy 160.02 80.01) (xy 152.654 80.01))
     (stroke (width 0) (type solid) (color 0 0 0 0))
   )
@@
     (stroke (width 0) (type solid) (color 0 0 0 0))
   )
+  (wire (pts (xy 175.006 121.666) (xy 186.944 121.666))
+    (stroke (width 0) (type solid) (color 0 0 0 0))
+  )
   (wire (pts (xy 176.53 80.01) (xy 176.53 85.09))
     (stroke (width 0) (type solid) (color 0 0 0 0))
@@
     (stroke (width 0) (type solid) (color 0 0 0 0))
   )
-  (wire (pts (xy 179.705 120.015) (xy 190.5 120.015))
+  (wire (pts (xy 186.944 121.666) (xy 186.944 120.904))
     (stroke (width 0) (type solid) (color 0 0 0 0))
   )
-  (wire (pts (xy 190.5 120.015) (xy 190.5 123.825))
+  (wire (pts (xy 186.944 121.666) (xy 186.944 122.428))
     (stroke (width 0) (type solid) (color 0 0 0 0))
   )
@@
     (effects (font (size 1.27 1.27)) (justify right bottom))
   )
-  (label "ground" (at 186.69 120.015 180)
+  (label "ground" (at 182.118 121.666 180)
     (effects (font (size 1.27 1.27)) (justify right bottom))
   )
@@
     (effects (font (size 1.27 1.27)) (justify right))
   )
-  (symbol (lib_id "power:+3V3") (at 148.59 76.2 0)
+  (symbol (lib_id "power:PWR_FLAG") (at 152.654 78.486 0) (unit 1)
     (in_bom yes) (on_board yes)
-    (property "Reference" "#PWR07" (id 0) (at 148.59 80.01 0)
+    (property "Reference" "#FLG?" (id 0) (at 152.654 76.581 0)
+      (effects (font (size 1.27 1.27)) hide)
+    )
+    (property "Value" "PWR_FLAG" (id 1) (at 153.416 73.66 0))
+    (property "Footprint" "" (id 2) (at 152.654 78.486 0)
+      (effects (font (size 1.27 1.27)) hide)
+    )
+    (property "Datasheet" "~" (id 3) (at 152.654 78.486 0)
+      (effects (font (size 1.27 1.27)) hide)
+    )
+  )
+  (symbol (lib_id "power:PWR_FLAG") (at 186.944 120.904 0) (unit 1)
+    (in_bom yes) (on_board yes)
+    (property "Reference" "#FLG?" (id 0) (at 186.944 118.999 0)
+      (effects (font (size 1.27 1.27)) hide)
+    )
+    (property "Value" "PWR_FLAG" (id 1) (at 186.944 115.57 0))
+    (property "Footprint" "" (id 2) (at 186.944 120.904 0)
+      (effects (font (size 1.27 1.27)) hide)
+    )
+    (property "Datasheet" "~" (id 3) (at 186.944 120.904 0)
+      (effects (font (size 1.27 1.27)) hide)
+    )
+  )
+  (symbol (lib_id "power:+3V3") (at 148.59 76.2 0) (unit 1)
+    (in_bom yes) (on_board yes)
+    (property "Reference" "#PWR05" (id 0) (at 148.59 80.01 0)
       (effects (font (size 1.27 1.27)) hide)
     )
@@
     )
   )
-  (symbol (lib_id "power:GND") (at 190.5 123.825 0)
+  (symbol (lib_id "power:GND") (at 186.944 122.428 0) (unit 1)
     (in_bom yes) (on_board yes)
-    (property "Reference" "#PWR08" (id 0) (at 190.5 130.175 0)
+    (property "Reference" "#PWR06" (id 0) (at 186.944 128.778 0)
       (effects (font (size 1.27 1.27)) hide)
     )
-    (property "Value" "GND" (id 1) (at 191.77 128.27 0))
-    (property "Footprint" "" (id 2) (at 190.5 123.825 0)
+    (property "Value" "GND" (id 1) (at 188.214 126.873 0))
+    (property "Footprint" "" (id 2) (at 186.944 122.428 0)
       (effects (font (size 1.27 1.27)) hide)
     )
-    (property "Datasheet" "" (id 3) (at 190.5 123.825 0)
+    (property "Datasheet" "" (id 3) (at 186.944 122.428 0)
       (effects (font (size 1.27 1.27)) hide)
     )
   )
-  (symbol (lib_id "Device:R") (at 163.83 80.01 90)
+  (symbol (lib_id "Device:R") (at 163.83 80.01 90) (unit 1)
     (in_bom yes) (on_board yes)
-    (property "Reference" "R2" (id 0) (at 164.465 73.66 90))
+    (property "Reference" "R1" (id 0) (at 164.465 73.66 90))
     (property "Value" "R" (id 1) (at 164.465 76.2 90))
     (property "Footprint" "Resistor_SMD:R_0805_2012Metric" (id 2) (at 163.83 81.788 90)
@@
     )
   )
-  (symbol (lib_id "Device:LED") (at 176.53 88.9 90)
+  (symbol (lib_id "Device:LED") (at 176.53 88.9 90) (unit 1)
     (in_bom yes) (on_board yes)
-    (property "Reference" "D2" (id 0) (at 180.34 88.9 90)
+    (property "Reference" "D1" (id 0) (at 180.34 88.9 90)
       (effects (font (size 1.27 1.27)) (justify right))
     )
@@
     )
   )
-  (symbol (lib_id "Device:Q_NMOS_DGS") (at 159.385 102.87 0)
+  (symbol (lib_id "Device:Q_NMOS_DGS") (at 159.385 102.87 0) (unit 1)
     (in_bom yes) (on_board yes)
-    (property "Reference" "Q2" (id 0) (at 165.1 102.235 0)
+    (property "Reference" "Q1" (id 0) (at 165.1 102.235 0)
       (effects (font (size 1.27 1.27)) (justify left))
     )
