File: led/led.kicad_sch (KiCad schematic)
At the start: 0 parts

Commit message: led
Connections:
- no-connect marks 0 -> 1
Other:
- added sheet led1 (led-sheet.kicad_sch)
Changed lines of the file:
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@@
 (kicad_sch (version 20201015) (generator eeschema)
   (paper "A4")
+  (no_connect (at 222.25 83.82))
   (sheet (at 168.91 60.96) (size 26.67 20.32)
     (stroke (width 0.001) (type solid) (color 132 0 132 1))
@@
     )
   )
+  (sheet (at 173.99 92.71) (size 26.67 20.32)
+    (stroke (width 0.001) (type solid) (color 132 0 132 1))
+    (fill (color 255 255 255 0.0000))
+    (property "Sheet name" "led1" (id 0) (at 173.99 92.0741 0)
+      (effects (font (size 1.27 1.27)) (justify left bottom))
+    )
+    (property "Sheet file" "led-sheet.kicad_sch" (id 1) (at 173.99 113.5389 0)
+      (effects (font (size 1.27 1.27)) (justify left top))
+    )
+    (pin "LED_A" input (at 173.99 97.79 180)
+      (effects (font (size 1.27 1.27)) (justify left))
+    )
+    (pin "LED_C" input (at 173.99 104.14 180)
+      (effects (font (size 1.27 1.27)) (justify left))
+    )
+  )
   (sheet_instances
     (path "/" (page "1"))
     (path "/f6f98991-c174-4124-bca3-675ab210d740/" (page "2"))
+    (path "/4dff663b-c177-47c1-8447-1314ace07df1/" (page ""))
   )
   (symbol_instances
@@
       (reference "TP2") (unit 1) (value "TestPoint") (footprint "TestPoint:TestPoint_Pad_1.0x1.0mm")
     )
+    (path "/4dff663b-c177-47c1-8447-1314ace07df1/6d1ae22a-56e7-4f68-8007-d9b1bbd2a6d1"
+      (reference "D2") (unit 1) (value "LED") (footprint "LED_SMD:LED_0805_2012Metric")
+    )
+    (path "/4dff663b-c177-47c1-8447-1314ace07df1/32c558c9-73c5-42f4-bab5-24c9340f9df1"
+      (reference "TP3") (unit 1) (value "TestPoint") (footprint "TestPoint:TestPoint_Pad_1.0x1.0mm")
+    )
+    (path "/4dff663b-c177-47c1-8447-1314ace07df1/39dd7655-a0be-4856-a0cf-d45a3e703a6a"
+      (reference "TP4") (unit 1) (value "TestPoint") (footprint "TestPoint:TestPoint_Pad_1.0x1.0mm")
+    )
   )

Commit message: sch
Connections:
- no-connect marks 1 -> 0
Other:
- removed sheet led1
Changed lines of the file:
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@@
 (kicad_sch (version 20201015) (generator eeschema)
   (paper "A4")
-  (no_connect (at 222.25 83.82))
-  (sheet (at 168.91 60.96) (size 26.67 20.32)
+  (sheet (at 245.11 132.08) (size 26.67 20.32)
     (stroke (width 0.001) (type solid) (color 132 0 132 1))
     (fill (color 255 255 255 0.0000))
-    (property "Sheet name" "led" (id 0) (at 168.91 60.3241 0)
+    (property "Sheet name" "led" (id 0) (at 245.11 131.4441 0)
       (effects (font (size 1.27 1.27)) (justify left bottom))
     )
-    (property "Sheet file" "led-sheet.kicad_sch" (id 1) (at 168.91 81.7889 0)
+    (property "Sheet file" "led-sheet.kicad_sch" (id 1) (at 245.11 152.9089 0)
       (effects (font (size 1.27 1.27)) (justify left top))
     )
-    (pin "LED_A" input (at 168.91 66.04 180)
+    (pin "LED_A" input (at 245.11 137.16 180)
       (effects (font (size 1.27 1.27)) (justify left))
     )
-    (pin "LED_C" input (at 168.91 72.39 180)
-      (effects (font (size 1.27 1.27)) (justify left))
-    )
-  )
-  (sheet (at 173.99 92.71) (size 26.67 20.32)
-    (stroke (width 0.001) (type solid) (color 132 0 132 1))
-    (fill (color 255 255 255 0.0000))
-    (property "Sheet name" "led1" (id 0) (at 173.99 92.0741 0)
-      (effects (font (size 1.27 1.27)) (justify left bottom))
-    )
-    (property "Sheet file" "led-sheet.kicad_sch" (id 1) (at 173.99 113.5389 0)
-      (effects (font (size 1.27 1.27)) (justify left top))
-    )
-    (pin "LED_A" input (at 173.99 97.79 180)
-      (effects (font (size 1.27 1.27)) (justify left))
-    )
-    (pin "LED_C" input (at 173.99 104.14 180)
-      (effects (font (size 1.27 1.27)) (justify left))
+    (pin "LED_C" input (at 271.78 143.51 0)
+      (effects (font (size 1.27 1.27)) (justify right))
     )
   )
@@
     (path "/" (page "1"))
     (path "/f6f98991-c174-4124-bca3-675ab210d740/" (page "2"))
-    (path "/4dff663b-c177-47c1-8447-1314ace07df1/" (page ""))
   )
   (symbol_instances
@@
       (reference "TP2") (unit 1) (value "TestPoint") (footprint "TestPoint:TestPoint_Pad_1.0x1.0mm")
     )
-    (path "/4dff663b-c177-47c1-8447-1314ace07df1/6d1ae22a-56e7-4f68-8007-d9b1bbd2a6d1"
-      (reference "D2") (unit 1) (value "LED") (footprint "LED_SMD:LED_0805_2012Metric")
-    )
-    (path "/4dff663b-c177-47c1-8447-1314ace07df1/32c558c9-73c5-42f4-bab5-24c9340f9df1"
-      (reference "TP3") (unit 1) (value "TestPoint") (footprint "TestPoint:TestPoint_Pad_1.0x1.0mm")
-    )
-    (path "/4dff663b-c177-47c1-8447-1314ace07df1/39dd7655-a0be-4856-a0cf-d45a3e703a6a"
-      (reference "TP4") (unit 1) (value "TestPoint") (footprint "TestPoint:TestPoint_Pad_1.0x1.0mm")
-    )
   )

Commit message: led
Other:
- added sheet led1 (led-sheet.kicad_sch)
- sheet led ports: added control; removed LED_A, LED_C
Changed lines of the file:
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@@
 (kicad_sch (version 20201015) (generator eeschema)
   (paper "A4")
-  (sheet (at 245.11 132.08) (size 26.67 20.32)
+  (wire (pts (xy 123.19 86.995) (xy 135.255 86.995))
+    (stroke (width 0) (type solid) (color 0 0 0 0))
+  )
+  (wire (pts (xy 123.19 90.805) (xy 123.19 86.995))
+    (stroke (width 0) (type solid) (color 0 0 0 0))
+  )
+  (wire (pts (xy 125.73 121.285) (xy 135.89 121.285))
+    (stroke (width 0) (type solid) (color 0 0 0 0))
+  )
+  (wire (pts (xy 125.73 122.555) (xy 125.73 121.285))
+    (stroke (width 0) (type solid) (color 0 0 0 0))
+  )
+  (symbol (lib_id "power:PWR_FLAG") (at 77.47 83.82 0) (unit 1)
+    (in_bom yes) (on_board yes)
+    (property "Reference" "#FLG01" (id 0) (at 77.47 81.915 0)
+      (effects (font (size 1.27 1.27)) hide)
+    )
+    (property "Value" "PWR_FLAG" (id 1) (at 78.105 78.74 0))
+    (property "Footprint" "" (id 2) (at 77.47 83.82 0)
+      (effects (font (size 1.27 1.27)) hide)
+    )
+    (property "Datasheet" "~" (id 3) (at 77.47 83.82 0)
+      (effects (font (size 1.27 1.27)) hide)
+    )
+  )
+  (symbol (lib_id "power:PWR_FLAG") (at 88.265 83.82 0) (unit 1)
+    (in_bom yes) (on_board yes)
+    (property "Reference" "#FLG02" (id 0) (at 88.265 81.915 0)
+      (effects (font (size 1.27 1.27)) hide)
+    )
+    (property "Value" "PWR_FLAG" (id 1) (at 88.9 78.74 0))
+    (property "Footprint" "" (id 2) (at 88.265 83.82 0)
+      (effects (font (size 1.27 1.27)) hide)
+    )
+    (property "Datasheet" "~" (id 3) (at 88.265 83.82 0)
+      (effects (font (size 1.27 1.27)) hide)
+    )
+  )
+  (symbol (lib_id "power:+3V3") (at 77.47 83.82 180) (unit 1)
+    (in_bom yes) (on_board yes)
+    (property "Reference" "#PWR01" (id 0) (at 77.47 80.01 0)
+      (effects (font (size 1.27 1.27)) hide)
+    )
+    (property "Value" "+3V3" (id 1) (at 77.47 88.9 0))
+    (property "Footprint" "" (id 2) (at 77.47 83.82 0)
+      (effects (font (size 1.27 1.27)) hide)
+    )
+    (property "Datasheet" "" (id 3) (at 77.47 83.82 0)
+      (effects (font (size 1.27 1.27)) hide)
+    )
+  )
+  (symbol (lib_id "power:GND") (at 88.265 83.82 0) (unit 1)
+    (in_bom yes) (on_board yes)
+    (property "Reference" "#PWR02" (id 0) (at 88.265 90.17 0)
+      (effects (font (size 1.27 1.27)) hide)
+    )
+    (property "Value" "GND" (id 1) (at 88.9 88.9 0))
+    (property "Footprint" "" (id 2) (at 88.265 83.82 0)
+      (effects (font (size 1.27 1.27)) hide)
+    )
+    (property "Datasheet" "" (id 3) (at 88.265 83.82 0)
+      (effects (font (size 1.27 1.27)) hide)
+    )
+  )
+  (symbol (lib_id "power:GND") (at 123.19 90.805 0) (unit 1)
+    (in_bom yes) (on_board yes)
+    (property "Reference" "#PWR03" (id 0) (at 123.19 97.155 0)
+      (effects (font (size 1.27 1.27)) hide)
+    )
+    (property "Value" "GND" (id 1) (at 123.825 95.885 0))
+    (property "Footprint" "" (id 2) (at 123.19 90.805 0)
+      (effects (font (size 1.27 1.27)) hide)
+    )
+    (property "Datasheet" "" (id 3) (at 123.19 90.805 0)
+      (effects (font (size 1.27 1.27)) hide)
+    )
+  )
+  (symbol (lib_id "power:GND") (at 125.73 122.555 0) (unit 1)
+    (in_bom yes) (on_board yes)
+    (property "Reference" "#PWR04" (id 0) (at 125.73 128.905 0)
+      (effects (font (size 1.27 1.27)) hide)
+    )
+    (property "Value" "GND" (id 1) (at 126.365 127.635 0))
+    (property "Footprint" "" (id 2) (at 125.73 122.555 0)
+      (effects (font (size 1.27 1.27)) hide)
+    )
+    (property "Datasheet" "" (id 3) (at 125.73 122.555 0)
+      (effects (font (size 1.27 1.27)) hide)
+    )
+  )
+  (sheet (at 135.255 81.915) (size 26.67 20.32)
     (stroke (width 0.001) (type solid) (color 132 0 132 1))
     (fill (color 255 255 255 0.0000))
-    (property "Sheet name" "led" (id 0) (at 245.11 131.4441 0)
+    (property "Sheet name" "led" (id 0) (at 135.255 81.2791 0)
       (effects (font (size 1.27 1.27)) (justify left bottom))
     )
-    (property "Sheet file" "led-sheet.kicad_sch" (id 1) (at 245.11 152.9089 0)
+    (property "Sheet file" "led-sheet.kicad_sch" (id 1) (at 135.255 102.7439 0)
       (effects (font (size 1.27 1.27)) (justify left top))
     )
-    (pin "LED_A" input (at 245.11 137.16 180)
+    (pin "control" input (at 135.255 86.995 180)
       (effects (font (size 1.27 1.27)) (justify left))
     )
-    (pin "LED_C" input (at 271.78 143.51 0)
-      (effects (font (size 1.27 1.27)) (justify right))
+  )
+  (sheet (at 135.89 116.205) (size 26.67 20.32)
+    (stroke (width 0.001) (type solid) (color 132 0 132 1))
+    (fill (color 255 255 255 0.0000))
+    (property "Sheet name" "led1" (id 0) (at 135.89 115.5691 0)
+      (effects (font (size 1.27 1.27)) (justify left bottom))
+    )
+    (property "Sheet file" "led-sheet.kicad_sch" (id 1) (at 135.89 137.0339 0)
+      (effects (font (size 1.27 1.27)) (justify left top))
+    )
+    (pin "control" input (at 135.89 121.285 180)
+      (effects (font (size 1.27 1.27)) (justify left))
     )
   )
@@
     (path "/" (page "1"))
     (path "/f6f98991-c174-4124-bca3-675ab210d740/" (page "2"))
+    (path "/dcad42d4-5b63-424b-86af-b88b9e20d7ef/" (page ""))
   )
   (symbol_instances
+    (path "/a1b6120d-76e3-4ade-9f03-b1aa363a5109"
+      (reference "#FLG01") (unit 1) (value "PWR_FLAG") (footprint "")
+    )
+    (path "/8434552a-da4e-4486-9c72-55d5df901d05"
+      (reference "#FLG02") (unit 1) (value "PWR_FLAG") (footprint "")
+    )
+    (path "/67f49fbf-1558-4b68-a072-1e33f31a3997"
+      (reference "#PWR01") (unit 1) (value "+3V3") (footprint "")
+    )
+    (path "/8ddd7777-9bc8-406e-8d03-52ced29ca5e5"
+      (reference "#PWR02") (unit 1) (value "GND") (footprint "")
+    )
+    (path "/532235a4-9431-4bd6-8e9f-eaf263e04563"
+      (reference "#PWR03") (unit 1) (value "GND") (footprint "")
+    )
+    (path "/b0b440e4-05c3-4ee9-83f7-4519142668a1"
+      (reference "#PWR04") (unit 1) (value "GND") (footprint "")
+    )
+    (path "/f6f98991-c174-4124-bca3-675ab210d740/301a2811-f3c7-43e4-b172-f5cfe8cfc596"
+      (reference "#PWR05") (unit 1) (value "+3V3") (footprint "")
+    )
+    (path "/f6f98991-c174-4124-bca3-675ab210d740/3f316cef-ed87-4764-8a96-2f74ba7f115b"
+      (reference "#PWR06") (unit 1) (value "GND") (footprint "")
+    )
     (path "/f6f98991-c174-4124-bca3-675ab210d740/6d1ae22a-56e7-4f68-8007-d9b1bbd2a6d1"
       (reference "D1") (unit 1) (value "LED") (footprint "LED_SMD:LED_0805_2012Metric")
     )
-    (path "/f6f98991-c174-4124-bca3-675ab210d740/32c558c9-73c5-42f4-bab5-24c9340f9df1"
-      (reference "TP1") (unit 1) (value "TestPoint") (footprint "TestPoint:TestPoint_Pad_1.0x1.0mm")
+    (path "/f6f98991-c174-4124-bca3-675ab210d740/a4b061e3-44cf-4957-b795-e75f05b2acf4"
+      (reference "Q1") (unit 1) (value "Q_NMOS_DGS") (footprint "Package_TO_SOT_SMD:SOT-23")
     )
-    (path "/f6f98991-c174-4124-bca3-675ab210d740/39dd7655-a0be-4856-a0cf-d45a3e703a6a"
-      (reference "TP2") (unit 1) (value "TestPoint") (footprint "TestPoint:TestPoint_Pad_1.0x1.0mm")
+    (path "/f6f98991-c174-4124-bca3-675ab210d740/a90b67b7-ebf2-4cee-be9b-2f504fc17d18"
+      (reference "R1") (unit 1) (value "R") (footprint "Resistor_SMD:R_0805_2012Metric")
+    )
+    (path "/dcad42d4-5b63-424b-86af-b88b9e20d7ef/301a2811-f3c7-43e4-b172-f5cfe8cfc596"
+      (reference "#PWR07") (unit 1) (value "+3V3") (footprint "")
+    )
+    (path "/dcad42d4-5b63-424b-86af-b88b9e20d7ef/3f316cef-ed87-4764-8a96-2f74ba7f115b"
+      (reference "#PWR08") (unit 1) (value "GND") (footprint "")
+    )
+    (path "/dcad42d4-5b63-424b-86af-b88b9e20d7ef/6d1ae22a-56e7-4f68-8007-d9b1bbd2a6d1"
+      (reference "D2") (unit 1) (value "LED") (footprint "LED_SMD:LED_0805_2012Metric")
+    )
+    (path "/dcad42d4-5b63-424b-86af-b88b9e20d7ef/a4b061e3-44cf-4957-b795-e75f05b2acf4"
+      (reference "Q2") (unit 1) (value "Q_NMOS_DGS") (footprint "Package_TO_SOT_SMD:SOT-23")
+    )
+    (path "/dcad42d4-5b63-424b-86af-b88b9e20d7ef/a90b67b7-ebf2-4cee-be9b-2f504fc17d18"
+      (reference "R2") (unit 1) (value "R") (footprint "Resistor_SMD:R_0805_2012Metric")
     )
   )

Commit message: net
Other:
- removed sheet led1
Changed lines of the file:
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@@
 (kicad_sch (version 20201015) (generator eeschema)
   (paper "A4")
-  (wire (pts (xy 123.19 86.995) (xy 135.255 86.995))
-    (stroke (width 0) (type solid) (color 0 0 0 0))
-  )
-  (wire (pts (xy 123.19 90.805) (xy 123.19 86.995))
-    (stroke (width 0) (type solid) (color 0 0 0 0))
-  )
-  (wire (pts (xy 125.73 121.285) (xy 135.89 121.285))
-    (stroke (width 0) (type solid) (color 0 0 0 0))
-  )
-  (wire (pts (xy 125.73 122.555) (xy 125.73 121.285))
-    (stroke (width 0) (type solid) (color 0 0 0 0))
-  )
-  (symbol (lib_id "power:PWR_FLAG") (at 77.47 83.82 0) (unit 1)
-    (in_bom yes) (on_board yes)
-    (property "Reference" "#FLG01" (id 0) (at 77.47 81.915 0)
-      (effects (font (size 1.27 1.27)) hide)
-    )
-    (property "Value" "PWR_FLAG" (id 1) (at 78.105 78.74 0))
-    (property "Footprint" "" (id 2) (at 77.47 83.82 0)
-      (effects (font (size 1.27 1.27)) hide)
-    )
-    (property "Datasheet" "~" (id 3) (at 77.47 83.82 0)
-      (effects (font (size 1.27 1.27)) hide)
-    )
-  )
-  (symbol (lib_id "power:PWR_FLAG") (at 88.265 83.82 0) (unit 1)
-    (in_bom yes) (on_board yes)
-    (property "Reference" "#FLG02" (id 0) (at 88.265 81.915 0)
-      (effects (font (size 1.27 1.27)) hide)
-    )
-    (property "Value" "PWR_FLAG" (id 1) (at 88.9 78.74 0))
-    (property "Footprint" "" (id 2) (at 88.265 83.82 0)
-      (effects (font (size 1.27 1.27)) hide)
-    )
-    (property "Datasheet" "~" (id 3) (at 88.265 83.82 0)
-      (effects (font (size 1.27 1.27)) hide)
-    )
-  )
-  (symbol (lib_id "power:+3V3") (at 77.47 83.82 180) (unit 1)
-    (in_bom yes) (on_board yes)
-    (property "Reference" "#PWR01" (id 0) (at 77.47 80.01 0)
-      (effects (font (size 1.27 1.27)) hide)
-    )
-    (property "Value" "+3V3" (id 1) (at 77.47 88.9 0))
-    (property "Footprint" "" (id 2) (at 77.47 83.82 0)
-      (effects (font (size 1.27 1.27)) hide)
-    )
-    (property "Datasheet" "" (id 3) (at 77.47 83.82 0)
-      (effects (font (size 1.27 1.27)) hide)
-    )
-  )
-  (symbol (lib_id "power:GND") (at 88.265 83.82 0) (unit 1)
-    (in_bom yes) (on_board yes)
-    (property "Reference" "#PWR02" (id 0) (at 88.265 90.17 0)
-      (effects (font (size 1.27 1.27)) hide)
-    )
-    (property "Value" "GND" (id 1) (at 88.9 88.9 0))
-    (property "Footprint" "" (id 2) (at 88.265 83.82 0)
-      (effects (font (size 1.27 1.27)) hide)
-    )
-    (property "Datasheet" "" (id 3) (at 88.265 83.82 0)
-      (effects (font (size 1.27 1.27)) hide)
-    )
-  )
-  (symbol (lib_id "power:GND") (at 123.19 90.805 0) (unit 1)
-    (in_bom yes) (on_board yes)
-    (property "Reference" "#PWR03" (id 0) (at 123.19 97.155 0)
-      (effects (font (size 1.27 1.27)) hide)
-    )
-    (property "Value" "GND" (id 1) (at 123.825 95.885 0))
-    (property "Footprint" "" (id 2) (at 123.19 90.805 0)
-      (effects (font (size 1.27 1.27)) hide)
-    )
-    (property "Datasheet" "" (id 3) (at 123.19 90.805 0)
-      (effects (font (size 1.27 1.27)) hide)
-    )
-  )
-  (symbol (lib_id "power:GND") (at 125.73 122.555 0) (unit 1)
-    (in_bom yes) (on_board yes)
-    (property "Reference" "#PWR04" (id 0) (at 125.73 128.905 0)
-      (effects (font (size 1.27 1.27)) hide)
-    )
-    (property "Value" "GND" (id 1) (at 126.365 127.635 0))
-    (property "Footprint" "" (id 2) (at 125.73 122.555 0)
-      (effects (font (size 1.27 1.27)) hide)
-    )
-    (property "Datasheet" "" (id 3) (at 125.73 122.555 0)
-      (effects (font (size 1.27 1.27)) hide)
-    )
-  )
   (sheet (at 135.255 81.915) (size 26.67 20.32)
     (stroke (width 0.001) (type solid) (color 132 0 132 1))
@@
     )
   )
-  (sheet (at 135.89 116.205) (size 26.67 20.32)
-    (stroke (width 0.001) (type solid) (color 132 0 132 1))
-    (fill (color 255 255 255 0.0000))
-    (property "Sheet name" "led1" (id 0) (at 135.89 115.5691 0)
-      (effects (font (size 1.27 1.27)) (justify left bottom))
-    )
-    (property "Sheet file" "led-sheet.kicad_sch" (id 1) (at 135.89 137.0339 0)
-      (effects (font (size 1.27 1.27)) (justify left top))
-    )
-    (pin "control" input (at 135.89 121.285 180)
-      (effects (font (size 1.27 1.27)) (justify left))
-    )
-  )
   (sheet_instances
     (path "/" (page "1"))
     (path "/f6f98991-c174-4124-bca3-675ab210d740/" (page "2"))
-    (path "/dcad42d4-5b63-424b-86af-b88b9e20d7ef/" (page ""))
   )
   (symbol_instances
-    (path "/a1b6120d-76e3-4ade-9f03-b1aa363a5109"
-      (reference "#FLG01") (unit 1) (value "PWR_FLAG") (footprint "")
-    )
-    (path "/8434552a-da4e-4486-9c72-55d5df901d05"
-      (reference "#FLG02") (unit 1) (value "PWR_FLAG") (footprint "")
-    )
-    (path "/67f49fbf-1558-4b68-a072-1e33f31a3997"
-      (reference "#PWR01") (unit 1) (value "+3V3") (footprint "")
-    )
-    (path "/8ddd7777-9bc8-406e-8d03-52ced29ca5e5"
-      (reference "#PWR02") (unit 1) (value "GND") (footprint "")
-    )
-    (path "/532235a4-9431-4bd6-8e9f-eaf263e04563"
-      (reference "#PWR03") (unit 1) (value "GND") (footprint "")
-    )
-    (path "/b0b440e4-05c3-4ee9-83f7-4519142668a1"
-      (reference "#PWR04") (unit 1) (value "GND") (footprint "")
-    )
     (path "/f6f98991-c174-4124-bca3-675ab210d740/301a2811-f3c7-43e4-b172-f5cfe8cfc596"
       (reference "#PWR05") (unit 1) (value "+3V3") (footprint "")
@@
       (reference "R1") (unit 1) (value "R") (footprint "Resistor_SMD:R_0805_2012Metric")
     )
-    (path "/dcad42d4-5b63-424b-86af-b88b9e20d7ef/301a2811-f3c7-43e4-b172-f5cfe8cfc596"
-      (reference "#PWR07") (unit 1) (value "+3V3") (footprint "")
-    )
-    (path "/dcad42d4-5b63-424b-86af-b88b9e20d7ef/3f316cef-ed87-4764-8a96-2f74ba7f115b"
-      (reference "#PWR08") (unit 1) (value "GND") (footprint "")
-    )
-    (path "/dcad42d4-5b63-424b-86af-b88b9e20d7ef/6d1ae22a-56e7-4f68-8007-d9b1bbd2a6d1"
-      (reference "D2") (unit 1) (value "LED") (footprint "LED_SMD:LED_0805_2012Metric")
-    )
-    (path "/dcad42d4-5b63-424b-86af-b88b9e20d7ef/a4b061e3-44cf-4957-b795-e75f05b2acf4"
-      (reference "Q2") (unit 1) (value "Q_NMOS_DGS") (footprint "Package_TO_SOT_SMD:SOT-23")
-    )
-    (path "/dcad42d4-5b63-424b-86af-b88b9e20d7ef/a90b67b7-ebf2-4cee-be9b-2f504fc17d18"
-      (reference "R2") (unit 1) (value "R") (footprint "Resistor_SMD:R_0805_2012Metric")
-    )
   )

Commit message: baseline
Changed lines of the file:
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@@
 (kicad_sch (version 20201015) (generator eeschema)
   (paper "A4")
-  (sheet (at 135.255 81.915) (size 26.67 20.32)
+  (sheet (at 151.765 78.105) (size 26.67 20.32)
     (stroke (width 0.001) (type solid) (color 132 0 132 1))
     (fill (color 255 255 255 0.0000))
-    (property "Sheet name" "led" (id 0) (at 135.255 81.2791 0)
+    (property "Sheet name" "led" (id 0) (at 151.765 77.4691 0)
       (effects (font (size 1.27 1.27)) (justify left bottom))
     )
-    (property "Sheet file" "led-sheet.kicad_sch" (id 1) (at 135.255 102.7439 0)
+    (property "Sheet file" "led-sheet.kicad_sch" (id 1) (at 151.765 98.9339 0)
       (effects (font (size 1.27 1.27)) (justify left top))
     )
-    (pin "control" input (at 135.255 86.995 180)
+    (pin "control" input (at 151.765 83.185 180)
       (effects (font (size 1.27 1.27)) (justify left))
     )
@@
   )
   (symbol_instances
+    (path "/f6f98991-c174-4124-bca3-675ab210d740/7c882403-2416-47bd-8142-e59dd72b85d2"
+      (reference "#FLG?") (unit 1) (value "PWR_FLAG") (footprint "")
+    )
+    (path "/f6f98991-c174-4124-bca3-675ab210d740/c3651b6a-2384-4d61-a9c6-16a6611a5d34"
+      (reference "#FLG?") (unit 1) (value "PWR_FLAG") (footprint "")
+    )
     (path "/f6f98991-c174-4124-bca3-675ab210d740/301a2811-f3c7-43e4-b172-f5cfe8cfc596"
       (reference "#PWR05") (unit 1) (value "+3V3") (footprint "")
