File: cap/cap.kicad_sch (KiCad schematic)
At the start: 3 parts

Commit message: cap
Parts:
- C1: value C -> 100u
Changed lines of the file:
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@@
       (effects (font (size 1.27 1.27)) (justify left))
     )
-    (property "Value" "C" (id 1) (at 149.86 77.47 0)
+    (property "Value" "100u" (id 1) (at 149.86 77.47 0)
       (effects (font (size 1.27 1.27)) (justify left))
     )
@@
   (symbol_instances
     (path "/88a958a5-1a43-4bdf-a829-8f7aace2cefd"
-      (reference "C1") (unit 1) (value "C") (footprint "Capacitor_SMD:C_0805_2012Metric")
+      (reference "C1") (unit 1) (value "100u") (footprint "Capacitor_SMD:C_0805_2012Metric")
     )
     (path "/9100811d-f90b-4a65-a37f-2871564a20b7"
