File: byhand/byhand.kicad_pcb (KiCad board)
At the start: 2 copper layers, 4 parts

Commit message: led
Parts:
- added R3: R, Resistor_SMD:R_0805_2012Metric, F.Cu at (165.0, 88.0)
- added R4: R, Resistor_SMD:R_0805_2012Metric, F.Cu at (164.0, 94.2)
Connections:
- net GND renamed ground
- D1 pad 1: /R_TOP -> /test
- R1 pad 1: /R_TOP -> /curlimit1/foo
- R2 pad 1: /LED_C -> /curlimit2/foo
Routing:
- net /R_TOP: track 9.70 -> 0.00 mm
- net /test: track 0.00 -> 5.87 mm
- net /LED_C: track 9.76 -> 4.92 mm
- net /curlimit2/foo: track 0.00 -> 3.02 mm
- net /curlimit1/foo: track 0.00 -> 2.03 mm
Other:
- board outline added: 17 x 17 mm
Changed lines of the file:
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@@
   (net 0 "")
   (net 1 "+3V3")
-  (net 2 "/R_TOP")
+  (net 2 "/test")
   (net 3 "/LED_C")
-  (net 4 "GND")
+  (net 4 "ground")
+  (net 5 "/curlimit1/foo")
+  (net 6 "/curlimit2/foo")
   (footprint "LED_SMD:LED_0805_2012Metric" (layer "F.Cu")
     (at 160 94.3)
@@
     )
   )
+  (footprint "Resistor_SMD:R_0805_2012Metric" (layer "F.Cu")
+    (at 164 94.195 180)
+    (descr "Resistor SMD 0805 (2012 Metric), square (rectangular) end terminal, IPC_7351 nominal, (Body size source: IPC-SM-782 page 72, https://www.pcb-3d.com/wordpress/wp-content/uploads/ipc-sm-782a_amendment_1_and_2.pdf), generated with kicad-footprint-generator")
+    (tags "resistor")
+    (property "Sheet file" "curlimit.kicad_sch")
+    (property "Sheet name" "curlimit2")
+    (attr smd)
+    (fp_text reference "R4" (at 0 -1.65) (layer "F.SilkS")
+      (effects (font (size 1 1) (thickness 0.15)))
+    )
+    (fp_text value "R" (at 0 1.65) (layer "F.Fab")
+      (effects (font (size 1 1) (thickness 0.15)))
+    )
+    (fp_text user "${REFERENCE}" (at 0 0) (layer "F.Fab")
+      (effects (font (size 0.5 0.5) (thickness 0.08)))
+    )
+    (fp_line (start -0.227064 -0.735) (end 0.227064 -0.735) (layer "F.SilkS") (width 0.12))
+    (fp_line (start -0.227064 0.735) (end 0.227064 0.735) (layer "F.SilkS") (width 0.12))
+    (fp_line (start 1.68 -0.95) (end 1.68 0.95) (layer "F.CrtYd") (width 0.05))
+    (fp_line (start -1.68 0.95) (end -1.68 -0.95) (layer "F.CrtYd") (width 0.05))
+    (fp_line (start -1.68 -0.95) (end 1.68 -0.95) (layer "F.CrtYd") (width 0.05))
+    (fp_line (start 1.68 0.95) (end -1.68 0.95) (layer "F.CrtYd") (width 0.05))
+    (fp_line (start -1 -0.625) (end 1 -0.625) (layer "F.Fab") (width 0.1))
+    (fp_line (start 1 0.625) (end -1 0.625) (layer "F.Fab") (width 0.1))
+    (fp_line (start 1 -0.625) (end 1 0.625) (layer "F.Fab") (width 0.1))
+    (fp_line (start -1 0.625) (end -1 -0.625) (layer "F.Fab") (width 0.1))
+    (pad "1" smd roundrect (at -0.9125 0 180) (size 1.025 1.4) (layers "F.Cu" "F.Paste" "F.Mask") (roundrect_rratio 0.243902)
+      (net 6 "/curlimit2/foo"))
+    (pad "2" smd roundrect (at 0.9125 0 180) (size 1.025 1.4) (layers "F.Cu" "F.Paste" "F.Mask") (roundrect_rratio 0.243902)
+      (net 3 "/LED_C"))
+    (model "${KISYS3DMOD}/Resistor_SMD.3dshapes/R_0805_2012Metric.wrl"
+      (offset (xyz 0 0 0))
+      (scale (xyz 1 1 1))
+      (rotate (xyz 0 0 0))
+    )
+  )
   (footprint "LED_SMD:LED_0805_2012Metric" (layer "F.Cu")
     (at 160 88)
@@
     (fp_line (start -1 -0.3) (end -1 0.6) (layer "F.Fab") (width 0.1))
     (pad "1" smd roundrect (at -0.9375 0) (size 0.975 1.4) (layers "F.Cu" "F.Paste" "F.Mask") (roundrect_rratio 0.25)
-      (net 2 "/R_TOP") (pinfunction "K"))
+      (net 2 "/test") (pinfunction "K"))
     (pad "2" smd roundrect (at 0.9375 0) (size 0.975 1.4) (layers "F.Cu" "F.Paste" "F.Mask") (roundrect_rratio 0.25)
       (net 1 "+3V3") (pinfunction "A"))
@@
   )
   (footprint "Resistor_SMD:R_0805_2012Metric" (layer "F.Cu")
+    (at 165 88 180)
+    (descr "Resistor SMD 0805 (2012 Metric), square (rectangular) end terminal, IPC_7351 nominal, (Body size source: IPC-SM-782 page 72, https://www.pcb-3d.com/wordpress/wp-content/uploads/ipc-sm-782a_amendment_1_and_2.pdf), generated with kicad-footprint-generator")
+    (tags "resistor")
+    (property "Sheet file" "curlimit.kicad_sch")
+    (property "Sheet name" "curlimit1")
+    (attr smd)
+    (fp_text reference "R3" (at 0 -1.65) (layer "F.SilkS")
+      (effects (font (size 1 1) (thickness 0.15)))
+    )
+    (fp_text value "R" (at 0 1.65) (layer "F.Fab")
+      (effects (font (size 1 1) (thickness 0.15)))
+    )
+    (fp_text user "${REFERENCE}" (at 0 0) (layer "F.Fab")
+      (effects (font (size 0.5 0.5) (thickness 0.08)))
+    )
+    (fp_line (start -0.227064 0.735) (end 0.227064 0.735) (layer "F.SilkS") (width 0.12))
+    (fp_line (start -0.227064 -0.735) (end 0.227064 -0.735) (layer "F.SilkS") (width 0.12))
+    (fp_line (start 1.68 0.95) (end -1.68 0.95) (layer "F.CrtYd") (width 0.05))
+    (fp_line (start 1.68 -0.95) (end 1.68 0.95) (layer "F.CrtYd") (width 0.05))
+    (fp_line (start -1.68 -0.95) (end 1.68 -0.95) (layer "F.CrtYd") (width 0.05))
+    (fp_line (start -1.68 0.95) (end -1.68 -0.95) (layer "F.CrtYd") (width 0.05))
+    (fp_line (start -1 -0.625) (end 1 -0.625) (layer "F.Fab") (width 0.1))
+    (fp_line (start -1 0.625) (end -1 -0.625) (layer "F.Fab") (width 0.1))
+    (fp_line (start 1 -0.625) (end 1 0.625) (layer "F.Fab") (width 0.1))
+    (fp_line (start 1 0.625) (end -1 0.625) (layer "F.Fab") (width 0.1))
+    (pad "1" smd roundrect (at -0.9125 0 180) (size 1.025 1.4) (layers "F.Cu" "F.Paste" "F.Mask") (roundrect_rratio 0.243902)
+      (net 5 "/curlimit1/foo"))
+    (pad "2" smd roundrect (at 0.9125 0 180) (size 1.025 1.4) (layers "F.Cu" "F.Paste" "F.Mask") (roundrect_rratio 0.243902)
+      (net 2 "/test"))
+    (model "${KISYS3DMOD}/Resistor_SMD.3dshapes/R_0805_2012Metric.wrl"
+      (offset (xyz 0 0 0))
+      (scale (xyz 1 1 1))
+      (rotate (xyz 0 0 0))
+    )
+  )
+  (footprint "Resistor_SMD:R_0805_2012Metric" (layer "F.Cu")
     (at 168.84 94.195)
     (descr "Resistor SMD 0805 (2012 Metric), square (rectangular) end terminal, IPC_7351 nominal, (Body size source: IPC-SM-782 page 72, https://www.pcb-3d.com/wordpress/wp-content/uploads/ipc-sm-782a_amendment_1_and_2.pdf), generated with kicad-footprint-generator")
@@
     (fp_line (start -1 0.625) (end -1 -0.625) (layer "F.Fab") (width 0.1))
     (pad "1" smd roundrect (at -0.9125 0) (size 1.025 1.4) (layers "F.Cu" "F.Paste" "F.Mask") (roundrect_rratio 0.243902)
-      (net 3 "/LED_C"))
+      (net 6 "/curlimit2/foo"))
     (pad "2" smd roundrect (at 0.9125 0) (size 1.025 1.4) (layers "F.Cu" "F.Paste" "F.Mask") (roundrect_rratio 0.243902)
-      (net 4 "GND"))
+      (net 4 "ground"))
     (model "${KISYS3DMOD}/Resistor_SMD.3dshapes/R_0805_2012Metric.wrl"
       (offset (xyz 0 0 0))
@@
     (fp_line (start 1 -0.625) (end 1 0.625) (layer "F.Fab") (width 0.1))
     (pad "1" smd roundrect (at -0.9125 0) (size 1.025 1.4) (layers "F.Cu" "F.Paste" "F.Mask") (roundrect_rratio 0.243902)
-      (net 2 "/R_TOP"))
+      (net 5 "/curlimit1/foo"))
     (pad "2" smd roundrect (at 0.9125 0) (size 1.025 1.4) (layers "F.Cu" "F.Paste" "F.Mask") (roundrect_rratio 0.243902)
-      (net 4 "GND"))
-    (model "${KISYS3DMOD}/Resistor_SMD.3dshapes/R_0805_2012Metric.wrl"
-      (offset (xyz 0 0 0))
-      (scale (xyz 1 1 1))
-      (rotate (xyz 0 0 0))
-    )
-  )
+      (net 4 "ground"))
+    (model "${KISYS3DMOD}/Resistor_SMD.3dshapes/R_0805_2012Metric.wrl"
+      (offset (xyz 0 0 0))
+      (scale (xyz 1 1 1))
+      (rotate (xyz 0 0 0))
+    )
+  )
+  (gr_line (start 156 97) (end 156 102) (layer "Edge.Cuts") (width 0.1))
+  (gr_line (start 173 102) (end 156 102) (layer "Edge.Cuts") (width 0.1))
+  (gr_line (start 156 97) (end 156 85) (layer "Edge.Cuts") (width 0.1))
+  (gr_line (start 156 85) (end 173 85) (layer "Edge.Cuts") (width 0.1))
+  (gr_line (start 173 97) (end 173 102) (layer "Edge.Cuts") (width 0.1))
+  (gr_line (start 173 85) (end 173 97) (layer "Edge.Cuts") (width 0.1))
   (segment (start 160.9375 88) (end 160.9375 94.3) (width 0.25) (layer "F.Cu") (net 1))
-  (segment (start 166.94749 86.97499) (end 167.9275 87.955) (width 0.25) (layer "F.Cu") (net 2))
-  (segment (start 159.0625 88) (end 160.08751 86.97499) (width 0.25) (layer "F.Cu") (net 2))
-  (segment (start 160.08751 86.97499) (end 166.94749 86.97499) (width 0.25) (layer "F.Cu") (net 2))
-  (segment (start 159.0625 94.3) (end 160.08751 95.32501) (width 0.25) (layer "F.Cu") (net 3))
-  (segment (start 160.08751 95.32501) (end 166.79749 95.32501) (width 0.25) (layer "F.Cu") (net 3))
-  (segment (start 166.79749 95.32501) (end 167.9275 94.195) (width 0.25) (layer "F.Cu") (net 3))
-  (segment (start 169.7525 87.955) (end 169.7525 94.195) (width 0.25) (layer "F.Cu") (net 4))
+  (segment (start 163.06249 86.97499) (end 160.08751 86.97499) (width 0.25) (layer "F.Cu") (net 2))
+  (segment (start 164.0875 88) (end 163.06249 86.97499) (width 0.25) (layer "F.Cu") (net 2))
+  (segment (start 160.08751 86.97499) (end 159.0625 88) (width 0.25) (layer "F.Cu") (net 2))
+  (segment (start 160.08751 95.32501) (end 159.0625 94.3) (width 0.25) (layer "F.Cu") (net 3))
+  (segment (start 163.0875 94.195) (end 161.95749 95.32501) (width 0.25) (layer "F.Cu") (net 3))
+  (segment (start 161.95749 95.32501) (end 160.08751 95.32501) (width 0.25) (layer "F.Cu") (net 3))
+  (segment (start 169.7525 94.195) (end 169.7525 87.955) (width 0.25) (layer "F.Cu") (net 4))
+  (segment (start 167.9275 87.955) (end 165.9575 87.955) (width 0.25) (layer "F.Cu") (net 5))
+  (segment (start 165.9575 87.955) (end 165.9125 88) (width 0.25) (layer "F.Cu") (net 5))
+  (segment (start 164.9125 94.195) (end 167.9275 94.195) (width 0.25) (layer "F.Cu") (net 6))
 )
