File: byhand/byhand.kicad_sch (KiCad schematic)
At the start: 0 parts

Commit message: led
Other:
- sheet curlimit1 ports: added test1; removed R_BOTTOM, R_TOP
- sheet curlimit2 ports: added test1; removed R_BOTTOM, R_TOP
- sheet led1 ports: added test; removed LED_A
- sheet led2 ports: added test; removed LED_A
Changed lines of the file:
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@@
 (kicad_sch (version 20201015) (generator eeschema)
   (paper "A4")
+  (junction (at 171.45 46.99) (diameter 0.9144) (color 0 0 0 0))
+  (wire (pts (xy 128.27 77.47) (xy 138.43 77.47))
+    (stroke (width 0) (type solid) (color 0 0 0 0))
+  )
   (wire (pts (xy 135.89 46.99) (xy 135.89 67.31))
     (stroke (width 0) (type solid) (color 0 0 0 0))
@@
     (stroke (width 0) (type solid) (color 0 0 0 0))
   )
-  (wire (pts (xy 138.43 74.93) (xy 138.43 80.01))
+  (wire (pts (xy 138.43 77.47) (xy 138.43 80.01))
     (stroke (width 0) (type solid) (color 0 0 0 0))
   )
@@
     (stroke (width 0) (type solid) (color 0 0 0 0))
   )
-  (wire (pts (xy 147.32 74.93) (xy 138.43 74.93))
-    (stroke (width 0) (type solid) (color 0 0 0 0))
-  )
   (wire (pts (xy 170.18 34.29) (xy 170.18 38.1))
     (stroke (width 0) (type solid) (color 0 0 0 0))
@@
     (stroke (width 0) (type solid) (color 0 0 0 0))
   )
+  (wire (pts (xy 170.18 46.99) (xy 171.45 46.99))
+    (stroke (width 0) (type solid) (color 0 0 0 0))
+  )
   (wire (pts (xy 171.45 46.99) (xy 171.45 67.31))
     (stroke (width 0) (type solid) (color 0 0 0 0))
@@
     (stroke (width 0) (type solid) (color 0 0 0 0))
   )
-  (wire (pts (xy 172.72 74.93) (xy 172.72 83.82))
-    (stroke (width 0) (type solid) (color 0 0 0 0))
-  )
   (wire (pts (xy 175.26 46.99) (xy 171.45 46.99))
-    (stroke (width 0) (type solid) (color 0 0 0 0))
-  )
-  (wire (pts (xy 175.26 74.93) (xy 172.72 74.93))
     (stroke (width 0) (type solid) (color 0 0 0 0))
   )
@@
     (effects (font (size 1.27 1.27)) (justify right bottom))
   )
+  (label "test" (at 138.43 46.99 180)
+    (effects (font (size 1.27 1.27)) (justify right bottom))
+  )
+  (global_label "ground" (shape input) (at 128.27 77.47 180)    (property "Intersheet References" "${INTERSHEET_REFS}" (id 0) (at 117.8015 77.3906 0)
+      (effects (font (size 1.27 1.27)) (justify right) hide)
+    )
+    (effects (font (size 1.27 1.27)) (justify right))
+  )
   (symbol (lib_id "power:PWR_FLAG") (at 222.25 25.4 0) (unit 1)
     (in_bom yes) (on_board yes)
@@
     )
   )
-  (symbol (lib_id "power:GND") (at 172.72 83.82 0) (unit 1)
-    (in_bom yes) (on_board yes)
-    (property "Reference" "#PWR04" (id 0) (at 172.72 90.17 0)
-      (effects (font (size 1.27 1.27)) hide)
-    )
-    (property "Value" "GND" (id 1) (at 173.99 88.9 0))
-    (property "Footprint" "" (id 2) (at 172.72 83.82 0)
-      (effects (font (size 1.27 1.27)) hide)
-    )
-    (property "Datasheet" "" (id 3) (at 172.72 83.82 0)
-      (effects (font (size 1.27 1.27)) hide)
-    )
-  )
   (symbol (lib_id "power:GND") (at 231.14 25.4 0) (unit 1)
     (in_bom yes) (on_board yes)
@@
       (effects (font (size 1.27 1.27)) (justify left top))
     )
-    (pin "R_TOP" input (at 147.32 67.31 180)
-      (effects (font (size 1.27 1.27)) (justify left))
-    )
-    (pin "R_BOTTOM" input (at 147.32 74.93 180)
+    (pin "test1" input (at 147.32 67.31 180)
       (effects (font (size 1.27 1.27)) (justify left))
     )
@@
       (effects (font (size 1.27 1.27)) (justify left top))
     )
-    (pin "R_TOP" input (at 175.26 67.31 180)
-      (effects (font (size 1.27 1.27)) (justify left))
-    )
-    (pin "R_BOTTOM" input (at 175.26 74.93 180)
+    (pin "test1" input (at 175.26 67.31 180)
       (effects (font (size 1.27 1.27)) (justify left))
     )
@@
       (effects (font (size 1.27 1.27)) (justify left top))
     )
-    (pin "LED_A" input (at 147.32 38.1 180)
+    (pin "test" input (at 147.32 38.1 180)
       (effects (font (size 1.27 1.27)) (justify left))
     )
@@
       (effects (font (size 1.27 1.27)) (justify left top))
     )
-    (pin "LED_A" input (at 175.26 38.1 180)
+    (pin "test" input (at 175.26 38.1 180)
       (effects (font (size 1.27 1.27)) (justify left))
     )
@@
       (reference "#PWR03") (unit 1) (value "+3V3") (footprint "")
     )
-    (path "/97cad436-5a7a-49f0-84ce-7ccc9397fa14"
-      (reference "#PWR04") (unit 1) (value "GND") (footprint "")
-    )
     (path "/9aa53e04-42ed-4963-ba66-e13debe8965d"
       (reference "#PWR0101") (unit 1) (value "+3V3") (footprint "")
@@
       (reference "R1") (unit 1) (value "R") (footprint "Resistor_SMD:R_0805_2012Metric")
     )
+    (path "/06532423-3d65-4f4e-90ea-5a7f8b79fbdb/35bfbc6a-2136-4c2d-bbb9-08f86a3ea32a"
+      (reference "R3") (unit 1) (value "R") (footprint "Resistor_SMD:R_0805_2012Metric")
+    )
     (path "/e43b63e9-cf5d-4959-8d2f-06eaf42d4980/a3187d92-a65f-466c-b2cb-1668b5181ab4"
       (reference "D2") (unit 1) (value "LED") (footprint "LED_SMD:LED_0805_2012Metric")
@@
       (reference "R2") (unit 1) (value "R") (footprint "Resistor_SMD:R_0805_2012Metric")
     )
-  )
+    (path "/736d39b2-e76b-4efe-a802-34234c19bc48/35bfbc6a-2136-4c2d-bbb9-08f86a3ea32a"
+      (reference "R4") (unit 1) (value "R") (footprint "Resistor_SMD:R_0805_2012Metric")
+    )
+  )
