File: byhand/curlimit.kicad_sch (KiCad schematic)
At the start: 1 part

Commit message: nice
Parts:
- renumbered R2 to R?
Changed lines of the file:
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@@
   (symbol (lib_id "Device:R") (at 151.13 86.36 0)
     (in_bom yes) (on_board yes)
-    (property "Reference" "R2" (id 0) (at 153.67 85.09 0)
+    (property "Reference" "R?" (id 0) (at 153.67 85.09 0)
       (effects (font (size 1.27 1.27)) (justify left))
     )

Commit message: pcb
Parts:
- R1: renamed from R?; footprint (none) -> Resistor_SMD:R_0805_2012Metric
Changed lines of the file:
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@@
   (symbol (lib_id "Device:R") (at 151.13 86.36 0)
     (in_bom yes) (on_board yes)
-    (property "Reference" "R?" (id 0) (at 153.67 85.09 0)
+    (property "Reference" "R1" (id 0) (at 153.67 85.09 0)
       (effects (font (size 1.27 1.27)) (justify left))
     )
@@
       (effects (font (size 1.27 1.27)) (justify left))
     )
-    (property "Footprint" "" (id 2) (at 149.352 86.36 90)
+    (property "Footprint" "Resistor_SMD:R_0805_2012Metric" (id 2) (at 149.352 86.36 90)
       (effects (font (size 1.27 1.27)) hide)
     )

Commit message: led
Parts:
- added R4: R, Resistor_SMD:R_0805_2012Metric, symbol Device:R
- renumbered R1 to R2
Connections:
- net R_BOTTOM renamed ground
- net R_TOP renamed foo
- net foo: now also R4.1
- new net test1: R4.2
Other:
- moved on the sheet: R2
Changed lines of the file:
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@@
 (kicad_sch (version 20201015) (generator eeschema)
   (paper "A4")
-  (wire (pts (xy 147.32 78.74) (xy 151.13 78.74))
+  (wire (pts (xy 171.45 91.44) (xy 173.99 91.44))
     (stroke (width 0) (type solid) (color 0 0 0 0))
   )
-  (wire (pts (xy 147.32 93.98) (xy 151.13 93.98))
+  (wire (pts (xy 173.99 76.835) (xy 189.23 76.835))
     (stroke (width 0) (type solid) (color 0 0 0 0))
   )
-  (wire (pts (xy 151.13 78.74) (xy 151.13 82.55))
+  (wire (pts (xy 173.99 82.55) (xy 173.99 76.835))
     (stroke (width 0) (type solid) (color 0 0 0 0))
   )
-  (wire (pts (xy 151.13 93.98) (xy 151.13 90.17))
+  (wire (pts (xy 173.99 91.44) (xy 173.99 90.17))
     (stroke (width 0) (type solid) (color 0 0 0 0))
   )
-  (hierarchical_label "R_TOP" (shape input) (at 147.32 78.74 180)
+  (wire (pts (xy 199.39 76.2) (xy 210.185 76.2))
+    (stroke (width 0) (type solid) (color 0 0 0 0))
+  )
+  (wire (pts (xy 217.805 76.2) (xy 232.41 76.2))
+    (stroke (width 0) (type solid) (color 0 0 0 0))
+  )
+  (label "foo" (at 179.705 76.835 180)
+    (effects (font (size 1.27 1.27)) (justify right bottom))
+  )
+  (label "foo" (at 206.375 76.2 180)
+    (effects (font (size 1.27 1.27)) (justify right bottom))
+  )
+  (global_label "ground" (shape input) (at 171.45 91.44 180)    (property "Intersheet References" "${INTERSHEET_REFS}" (id 0) (at 160.9815 91.3606 0)
+      (effects (font (size 1.27 1.27)) (justify right) hide)
+    )
     (effects (font (size 1.27 1.27)) (justify right))
   )
-  (hierarchical_label "R_BOTTOM" (shape input) (at 147.32 93.98 180)
-    (effects (font (size 1.27 1.27)) (justify right))
+  (hierarchical_label "test1" (shape input) (at 232.41 76.2 0)
+    (effects (font (size 1.27 1.27)) (justify left))
   )
-  (symbol (lib_id "Device:R") (at 151.13 86.36 0)
+  (symbol (lib_id "Device:R") (at 173.99 86.36 0)
     (in_bom yes) (on_board yes)
-    (property "Reference" "R1" (id 0) (at 153.67 85.09 0)
+    (property "Reference" "R2" (id 0) (at 176.53 85.09 0)
       (effects (font (size 1.27 1.27)) (justify left))
     )
-    (property "Value" "R" (id 1) (at 153.67 87.63 0)
+    (property "Value" "R" (id 1) (at 176.53 87.63 0)
       (effects (font (size 1.27 1.27)) (justify left))
     )
-    (property "Footprint" "Resistor_SMD:R_0805_2012Metric" (id 2) (at 149.352 86.36 90)
+    (property "Footprint" "Resistor_SMD:R_0805_2012Metric" (id 2) (at 172.212 86.36 90)
       (effects (font (size 1.27 1.27)) hide)
     )
-    (property "Datasheet" "~" (id 3) (at 151.13 86.36 0)
+    (property "Datasheet" "~" (id 3) (at 173.99 86.36 0)
       (effects (font (size 1.27 1.27)) hide)
     )
+  )
+  (symbol (lib_id "Device:R") (at 213.995 76.2 90)
+    (in_bom yes) (on_board yes)
+    (property "Reference" "R4" (id 0) (at 212.725 73.66 0)
+      (effects (font (size 1.27 1.27)) (justify left))
+    )
+    (property "Value" "R" (id 1) (at 215.265 73.66 0)
+      (effects (font (size 1.27 1.27)) (justify left))
+    )
+    (property "Footprint" "Resistor_SMD:R_0805_2012Metric" (id 2) (at 213.995 77.978 90)
+      (effects (font (size 1.27 1.27)) hide)
+    )
+    (property "Datasheet" "~" (id 3) (at 213.995 76.2 0)
+      (effects (font (size 1.27 1.27)) hide)
+    )
