File: byhand/led.kicad_sch (KiCad schematic)
At the start: 1 part

Commit message: nice
Parts:
- renumbered D2 to D?
Changed lines of the file:
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@@
   (symbol (lib_id "Device:LED") (at 144.78 81.28 90)
     (in_bom yes) (on_board yes)
-    (property "Reference" "D2" (id 0) (at 148.59 81.28 90)
+    (property "Reference" "D?" (id 0) (at 148.59 81.28 90)
       (effects (font (size 1.27 1.27)) (justify right))
     )

Commit message: pcb
Parts:
- D1: renamed from D?; footprint (none) -> LED_SMD:LED_0805_2012Metric
Changed lines of the file:
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@@
   (symbol (lib_id "Device:LED") (at 144.78 81.28 90)
     (in_bom yes) (on_board yes)
-    (property "Reference" "D?" (id 0) (at 148.59 81.28 90)
+    (property "Reference" "D1" (id 0) (at 148.59 81.28 90)
       (effects (font (size 1.27 1.27)) (justify right))
     )
@@
       (effects (font (size 1.27 1.27)) (justify right))
     )
-    (property "Footprint" "" (id 2) (at 144.78 81.28 0)
+    (property "Footprint" "LED_SMD:LED_0805_2012Metric" (id 2) (at 144.78 81.28 0)
       (effects (font (size 1.27 1.27)) hide)
     )

Commit message: led
Parts:
- renumbered D1 to D2
Connections:
- net LED_A renamed test
Changed lines of the file:
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@@
 (kicad_sch (version 20201015) (generator eeschema)
   (paper "A4")
-  (wire (pts (xy 138.43 76.2) (xy 144.78 76.2))
+  (wire (pts (xy 124.46 76.2) (xy 144.78 76.2))
     (stroke (width 0) (type solid) (color 0 0 0 0))
   )
@@
     (stroke (width 0) (type solid) (color 0 0 0 0))
   )
-  (hierarchical_label "LED_A" (shape input) (at 138.43 76.2 180)
+  (hierarchical_label "test" (shape input) (at 124.46 76.2 180)
     (effects (font (size 1.27 1.27)) (justify right))
   )
@@
   (symbol (lib_id "Device:LED") (at 144.78 81.28 90)
     (in_bom yes) (on_board yes)
-    (property "Reference" "D1" (id 0) (at 148.59 81.28 90)
+    (property "Reference" "D2" (id 0) (at 148.59 81.28 90)
       (effects (font (size 1.27 1.27)) (justify right))
     )
